File: PCB/Button PCB/procon_button_board.kicad_pcb (KiCad board)
At the start: 4 copper layers, 109.4 x 54.3 mm, 33 parts, among them J1 To Button Board, J2 bumpers, SW1 TL3315NF100Q, SW10 DPAD, SW11 DPAD, SW12 DPAD, SW2 TL3315NF100Q, SW3 TL3315NF100Q, SW4 TL3315NF100Q, SW5 BPAD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

Commit message: Update with split dpad file test
Other:
- board text added: "ProCon Button Board Designed by Mitch"
- board text removed: "ProGCC 3 Button Board Designed by Mitch"
Changed lines of the file:
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@@
       (drillshape 0)
       (scaleselection 1)
-      (outputdirectory "production/drill")
+      (outputdirectory "production/gerber/")
     )
   )
@@
     (property "Sheetname" "")
     (attr smd)
-    (fp_text reference "SW4" (at 0 2.9972 unlocked) (layer "F.SilkS")
+    (fp_text reference "SW4" (at 4.096 0.108 unlocked) (layer "F.SilkS")
         (effects (font (size 1 1) (thickness 0.1)))
     )
@@
     (property "Sheetname" "")
     (attr smd)
-    (fp_text reference "SW2" (at 0 2.9972 unlocked) (layer "F.SilkS")
+    (fp_text reference "SW2" (at 2.646 2.658 unlocked) (layer "F.SilkS")
         (effects (font (size 1 1) (thickness 0.1)))
     )
@@
     (property "Sheetname" "")
     (attr smd)
-    (fp_text reference "SW1" (at 0 2.9972 unlocked) (layer "F.SilkS")
+    (fp_text reference "SW1" (at -3.229 2.608 unlocked) (layer "F.SilkS")
         (effects (font (size 1 1) (thickness 0.1)))
     )
@@
     (property "Sheetname" "")
     (attr smd)
-    (fp_text reference "L9" (at 1.016 2.032 unlocked) (layer "F.SilkS")
+    (fp_text reference "L9" (at 1.816 1.848 unlocked) (layer "F.SilkS")
         (effects (font (size 1 1) (thickness 0.15)))
     )
@@
     (property "Sheetname" "")
     (attr smd)
-    (fp_text reference "L7" (at 1.016 2.032 unlocked) (layer "F.SilkS")
+    (fp_text reference "L7" (at -2.154 0.483 unlocked) (layer "F.SilkS")
         (effects (font (size 1 1) (thickness 0.15)))
     )
@@
     (property "Sheetname" "")
     (attr smd)
-    (fp_text reference "SW3" (at 0 2.9972 unlocked) (layer "F.SilkS")
+    (fp_text reference "SW3" (at 4.121 -0.017 unlocked) (layer "F.SilkS")
         (effects (font (size 1 1) (thickness 0.1)))
     )
@@
     (property "ki_keywords" "diode")
     (attr smd)
-    (fp_text reference "D2" (at 0 2 270) (layer "B.SilkS")
+    (fp_text reference "D2" (at 2.615612 -0.25572 270) (layer "B.SilkS")
         (effects (font (size 1 1) (thickness 0.15)) (justify mirror))
     )
@@
     (property "ki_keywords" "diode")
     (attr smd)
-    (fp_text reference "D5" (at 0 2 270) (layer "B.SilkS")
+    (fp_text reference "D5" (at 2.640612 0.63828 270) (layer "B.SilkS")
         (effects (font (size 1 1) (thickness 0.15)) (justify mirror))
     )
@@
     (property "ki_keywords" "diode")
     (attr smd)
-    (fp_text reference "D4" (at 0 2 270) (layer "B.SilkS")
+    (fp_text reference "D4" (at 2.540612 0.49028 270) (layer "B.SilkS")
         (effects (font (size 1 1) (thickness 0.15)) (justify mirror))
     )
@@
     (property "ki_keywords" "diode")
     (attr smd)
-    (fp_text reference "D6" (at 0 2 270) (layer "B.SilkS")
+    (fp_text reference "D6" (at 2.715612 -0.11372 270) (layer "B.SilkS")
         (effects (font (size 1 1) (thickness 0.15)) (justify mirror))
     )
@@
     (property "ki_keywords" "diode")
     (attr smd)
-    (fp_text reference "D3" (at 0 2 270) (layer "B.SilkS")
+    (fp_text reference "D3" (at 2.590612 -0.55772 270) (layer "B.SilkS")
         (effects (font (size 1 1) (thickness 0.15)) (justify mirror))
     )
@@
     (property "ki_keywords" "diode")
     (attr smd)
-    (fp_text reference "D1" (at 0 2 270) (layer "B.SilkS")
+    (fp_text reference "D1" (at 2.415612 0.34628 270) (layer "B.SilkS")
         (effects (font (size 1 1) (thickness 0.15)) (justify mirror))
     )
@@
   (gr_line (start 187.848 112.496) (end 170.198 112.496)
     (stroke (width 0.1) (type solid)) (layer "Edge.Cuts"))
-  (gr_text "ProGCC 3\nButton Board\nDesigned by Mitch" (at 105.664 166.37) (layer "F.SilkS")
+  (gr_text "ProCon\nButton Board\nDesigned by Mitch" (at 105.664 166.37) (layer "F.SilkS")
     (effects (font (size 0.65 0.65) (thickness 0.15)) (justify left bottom))
   )
