File: PCB/Button PCB RGB/procon_button_board.kicad_pcb (KiCad board)
At the start: 4 copper layers, 109.4 x 54.3 mm, 34 parts, among them J1 To Button Board, J2 bumpers, J3 bumpers, SW1 TL3315NF100Q, SW10 DPAD, SW11 DPAD, SW12 DPAD, SW2 TL3315NF100Q, SW3 TL3315NF100Q, SW4 TL3315NF100Q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

Commit message: Update component BOM and production files.
Parts:
- added L13: SK6805-EC-10, hhl:SK6805-EC-10, F.Cu at (153.7, 125.0)
- SW10, SW11, SW12, SW9: footprint progcc_v3:progcc_dpad -> hhl:ring_dpad
- SW5, SW6, SW7, SW8: footprint progcc_v3:progcc_bpad -> hhl:ring_pad
- moved J3 0.49 mm to (190.5, 147.8)
- turned SW10 to 90 degrees
- turned SW11 to 180 degrees
- turned SW12 to -90 degrees
- turned SW5 to 180 degrees
- turned SW6 to 180 degrees
- turned SW7 to 180 degrees
- turned SW8 to 180 degrees
- turned SW9 to 0 degrees
Connections:
- net Net-(L6-DOUT) renamed L_HOME
Routing:
- net Scan_A: track 168.1 -> 217.6 mm, vias 7 -> 11
- net GND: track 42.7 -> 68.7 mm, vias 34 -> 41
- net L_HOME: track 21.3 -> 34.4 mm, vias 0 -> 2
- net DU_Pull: track 50.3 -> 62.8 mm, vias 4 -> 5
- net DR_Pull: track 20.1 -> 32.1 mm
- net DD_Pull: track 34.4 -> 44.1 mm
- net Scan_B: track 93.5 -> 85.9 mm, vias 11 -> 8
- net DL_Pull: track 42.2 -> 47.2 mm, vias 6 -> 7
- net +3V3: track 36.5 -> 39.3 mm, vias 13 -> 14
- net X_Pull: track 83.2 -> 81.6 mm
- net B_Pull: track 93.0 -> 91.6 mm
- net Net-(L10-DIN): track 20.6 -> 21.9 mm
Other:
- board text added: "ProCon Button Board 3.2 Designed by Mitch"
- board text removed: "ProCon Button Board Designed by Mitch"
