File: PCB/Button PCB RGB/procon_button_board.kicad_sch (KiCad schematic)
At the start: 33 parts, among them J1 To Button Board, J2 bumpers, J3 bumpers, SW1 TL3315NF100Q, SW10 DPAD, SW11 DPAD, SW12 DPAD, SW2 TL3315NF100Q, SW3 TL3315NF100Q, SW4 TL3315NF100Q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

Commit message: Update component BOM and production files.
Parts:
- added L13: SK6805-EC-10, hhl:SK6805-EC-10, symbol hhl:SK6805-EC-10
- D1, D2, D3, D4, D5, D6: MPN (none) -> BAS16VY,115
- J1: MPN (none) -> molex_5051101492_14P
- L1, L10, L11, L12, L2, L3, L4, L5, L6, L7, L8, L9: MPN (none) -> SK6805-EC-10
- SW10, SW11, SW12, SW9: footprint progcc_v3:progcc_dpad -> hhl:ring_dpad; now not fitted
- SW5, SW6, SW7, SW8: footprint progcc_v3:progcc_bpad -> hhl:ring_pad; now not fitted
Connections:
- net +3V3: now also L13.2 (VDD)
- net GND: now also L13.4 (GND)
- net L_HOME: now reaches L6.3 (DOUT), L7.1 (DIN)
- net L_HOME: now also L13.1 (DIN)
Other:
- note added: "Secondary Home LED"

Commit message: Update production files
Parts:
- D1, D2, D3, D4, D5, D6: LCSC (none) -> C135826; Package (none) -> SOT-363
- J1: LCSC (none) -> C3169593; MPN molex_5051101492_14P -> 5051101492; Package (none) -> SMD,P=0.5mm,Surface Mount，Right Angle
- J2, J3: LCSC (none) -> C5527934; MPN molex_5034800540 -> 5034800540; Package (none) -> -
- L1, L10, L11, L12, L13, L2, L3, L4, L5, L6, L7, L8, L9: Package (none) -> SK6805-EC-10
- SW1, SW2, SW3, SW4: value TL3315NF100Q -> PTS540JM035SMTRLFS; LCSC (none) -> C221864; Link (none) -> https://www.lcsc.com/product-detail/Tactile-Switches_C-K-PT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; Package (none) -> SMD,3.7x3.7mm
Other:
- company: HHL/Esca -> Hand Held Legend, LLC
- title: ProGCC v3 Button Board -> ProGCC V3 Button PCB
