File: PCB/Battery PCB/procon_battery_pcb.kicad_sch (KiCad schematic)
At the start: 2 parts, among them J1 Conn_01x04_Pin, U1 1982633-1

Commit message: Update component BOM and production files.
Parts:
- U1: MPN (none) -> 1982633-1; Price (none) -> 1.08

Commit message: Update production files
Parts:
- U1: LCSC (none) -> C5877665; Link (none) -> https://www.lcsc.com/product-detail/BatteryConnector_TE-Con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; Package (none) -> -
Other:
- company: (none) -> Hand Held Legend, LLC
- title: (none) -> ProCon Battery PCB
Changed lines of the file:
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@@
 	(generator_version "8.0")
 	(paper "User" 135.001 89.9922)
+	(title_block
+		(title "ProCon Battery PCB")
+		(date "2024-10-29")
+		(company "Hand Held Legend, LLC")
+		(comment 1 "Designed by Mitch Cairns")
+	)
 	(wire
 		(pts
@@
 			)
 		)
-		(property "Description" ""
+		(property "Description" "BatteryConnector"
 			(at 39.37 26.67 0)
 			(effects
@@
 		)
 		(property "Price" "1.08"
+			(at 39.37 26.67 0)
+			(effects
+				(font
+					(size 1.27 1.27)
+				)
+				(hide yes)
+			)
+		)
+		(property "LCSC" "C5877665"
+			(at 39.37 26.67 0)
+			(effects
+				(font
+					(size 1.27 1.27)
+				)
+				(hide yes)
+			)
+		)
+		(property "Link" "https://www.lcsc.com/product-detail/BatteryConnector_TE-Connectivity-1982633-1_C5877665.html"
+			(at 39.37 26.67 0)
+			(effects
+				(font
+					(size 1.27 1.27)
+				)
+				(hide yes)
+			)
+		)
+		(property "Package" "-"
 			(at 39.37 26.67 0)
 			(effects
@@
 			(at 63.5 26.67 0)
 			(effects
+				(font
+					(size 1.27 1.27)
+				)
+				(hide yes)
+			)
+		)
+		(property "LCSC" ""
+			(at 63.5 26.67 0)
+			(effects
+				(font
+					(size 1.27 1.27)
+				)
+				(hide yes)
+			)
+		)
+		(property "Link" ""
+			(at 63.5 26.67 0)
+			(effects
+				(font
+					(size 1.27 1.27)
+				)
+				(hide yes)
+			)
+		)
+		(property "Package" ""
+			(at 63.5 26.67 0)
+			(effects
