File: PCB/Trigger Button PCB RGB/procon_trigger_pcb.kicad_sch (KiCad schematic)
At the start: 10 parts, among them J1 Conn_01x05_Pin, J2 Conn_01x05_Pin, SW1 SW_Push, SW2 SW_Push, SW3 SW_Push, SW4 SW_Push

Commit message: Update component BOM and production files.
Parts:
- J1, J2, SW1, SW2, SW3, SW4: now not fitted

Commit message: Update production files
Parts:
- J1, J2: LCSC (none) -> -; Link (none) -> -; MPN (none) -> -; Package (none) -> -
- L1, L2, L3, L4: Package (none) -> SK6805-EC-10
Other:
- company: (none) -> Hand Held Legend, LLC
- title: (none) -> ProGCC RGB Trigger Flex PCB
